Commit message: msg

File: hand/robots/sr_hand_bimanual.urdf (robot description, URDF)
Before this commit: robot bimanual_shadowhand_motor, 65 links, 64 joints
Links:
- link lh_ffdistal: mass 0.012 -> None
- link lh_ffknuckle: mass 0.008 -> None
- link lh_ffmiddle: mass 0.017 -> None
- link lh_ffproximal: mass 0.030 -> None
- link lh_fftip: mass 0.001 -> None
- link lh_forearm: mass 3.0 -> None
- link lh_lfdistal: mass 0.012 -> None
- link lh_lfknuckle: mass 0.008 -> None
- link lh_lfmetacarpal: mass 0.030 -> None
- link lh_lfmiddle: mass 0.017 -> None
- link lh_lfproximal: mass 0.030 -> None
- link lh_lftip: mass 0.001 -> None
- link lh_mfdistal: mass 0.012 -> None
- link lh_mfknuckle: mass 0.008 -> None
- link lh_mfmiddle: mass 0.017 -> None
- link lh_mfproximal: mass 0.030 -> None
- link lh_mftip: mass 0.001 -> None
- link lh_palm: mass 0.3 -> None
- link lh_rfdistal: mass 0.012 -> None
- link lh_rfknuckle: mass 0.008 -> None
- link lh_rfmiddle: mass 0.017 -> None
- link lh_rfproximal: mass 0.030 -> None
- link lh_rftip: mass 0.001 -> None
- link lh_thbase: mass 0.010 -> None
- link lh_thdistal: mass 0.016 -> None
- link lh_thhub: mass 0.005 -> None
- link lh_thmiddle: mass 0.020 -> None
- link lh_thproximal: mass 0.040 -> None
- link lh_thtip: mass 0.001 -> None
- link lh_wrist: mass 0.1 -> None
- link rh_ffdistal: mass 0.012 -> None
- link rh_ffknuckle: mass 0.008 -> None
- link rh_ffmiddle: mass 0.017 -> None
- link rh_ffproximal: mass 0.030 -> None
- link rh_fftip: mass 0.001 -> None
- link rh_forearm: mass 3.0 -> None
- link rh_lfdistal: mass 0.012 -> None
- link rh_lfknuckle: mass 0.008 -> None
- link rh_lfmetacarpal: mass 0.030 -> None
- link rh_lfmiddle: mass 0.017 -> None
- link rh_lfproximal: mass 0.030 -> None
- link rh_lftip: mass 0.001 -> None
- link rh_mfdistal: mass 0.012 -> None
- link rh_mfknuckle: mass 0.008 -> None
- link rh_mfmiddle: mass 0.017 -> None
- link rh_mfproximal: mass 0.030 -> None
- link rh_mftip: mass 0.001 -> None
- link rh_palm: mass 0.3 -> None
- link rh_rfdistal: mass 0.012 -> None
- link rh_rfknuckle: mass 0.008 -> None
- link rh_rfmiddle: mass 0.017 -> None
- link rh_rfproximal: mass 0.030 -> None
- link rh_rftip: mass 0.001 -> None
- link rh_thbase: mass 0.010 -> None
- link rh_thdistal: mass 0.016 -> None
- link rh_thhub: mass 0.005 -> None
- link rh_thmiddle: mass 0.020 -> None
- link rh_thproximal: mass 0.040 -> None
- link rh_thtip: mass 0.001 -> None
- link rh_wrist: mass 0.1 -> None
