Commit message: m

File: hand/xacro/wrist/wrist.urdf.xacro (robot description, xacro)
@@ -36,5 +36,5 @@
         <origin xyz="0 0 0" rpy="0 0 0" />
         <geometry name="${prefix}wrist_visual">
-          <mesh filename="package://sr_description/meshes/components/wrist/wrist_${hand_version}.dae"
+          <mesh filename="package://botdylan/meshes/components/wrist/wrist_${hand_version}.dae"
           scale="${reflect*0.001} 0.001 0.001" />
         </geometry>

File: robots/sr_hand.urdf (robot description, URDF)
Before this commit: robot shadowhand_motor, 33 links, 32 joints
Links:
- link rh_ffdistal: geometry collision mesh filename=package://botdylan/meshes/components/f_distal/pst/f_distal_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 scale=0.001 0.001 0.001; visual mesh filename=package://botdylan/meshes/components/f_distal/pst/f_distal_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 scale=0.001 0.001 0.001
- link rh_ffknuckle: geometry collision cylinder length=0.014 radius=0.007; visual mesh filename=package://botdylan/meshes/components/f_knuckle/f_knuckle_E3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 scale=0.001 0.001 0.001
- link rh_ffmiddle: geometry collision cylinder length=0.025 radius=0.007; collision sphere radius=0.007
- link rh_ffproximal: geometry collision cylinder length=0.040 radius=0.007; visual mesh filename=package://botdylan/meshes/components/f_proximal/f_proximal_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 scale=0.001 0.001 0.001
- link rh_forearm: geometry collision box size=0.07 0.07 0.07; collision mesh filename=package://botdylan/meshes/components/forearm/forearm_collis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 scale=0.001 0.001 0.001
- link rh_lfdistal: geometry collision mesh filename=package://botdylan/meshes/components/f_distal/pst/f_distal_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 scale=0.001 0.001 0.001; visual mesh filename=package://botdylan/meshes/components/f_distal/pst/f_distal_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 scale=0.001 0.001 0.001
- link rh_lfknuckle: geometry collision cylinder length=0.014 radius=0.007; visual mesh filename=package://botdylan/meshes/components/f_knuckle/f_knuckle_E3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 scale=0.001 0.001 0.001
- link rh_lfmetacarpal: geometry collision box size=0.018 0.024 0.040; visual mesh filename=package://botdylan/meshes/components/lf_metacarpal/lf_metac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 scale=0.001 0.001 0.001
- link rh_lfmiddle: geometry collision cylinder length=0.025 radius=0.007; collision sphere radius=0.007
- link rh_lfproximal: geometry collision cylinder length=0.040 radius=0.007; visual mesh filename=package://botdylan/meshes/components/f_proximal/f_proximal_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 scale=0.001 0.001 0.001
- link rh_mfdistal: geometry collision mesh filename=package://botdylan/meshes/components/f_distal/pst/f_distal_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 scale=0.001 0.001 0.001; visual mesh filename=package://botdylan/meshes/components/f_distal/pst/f_distal_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 scale=0.001 0.001 0.001
- link rh_mfknuckle: geometry collision cylinder length=0.014 radius=0.007; visual mesh filename=package://botdylan/meshes/components/f_knuckle/f_knuckle_E3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 scale=0.001 0.001 0.001
- link rh_mfmiddle: geometry collision cylinder length=0.025 radius=0.007; collision sphere radius=0.007
- link rh_mfproximal: geometry collision cylinder length=0.040 radius=0.007; visual mesh filename=package://botdylan/meshes/components/f_proximal/f_proximal_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 scale=0.001 0.001 0.001
- link rh_palm: geometry collision box size=0.018 0.024 0.004; collision box size=0.020 0.024 0.040
- link rh_rfdistal: geometry collision mesh filename=package://botdylan/meshes/components/f_distal/pst/f_distal_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 scale=0.001 0.001 0.001; visual mesh filename=package://botdylan/meshes/components/f_distal/pst/f_distal_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 scale=0.001 0.001 0.001
- link rh_rfknuckle: geometry collision cylinder length=0.014 radius=0.007; visual mesh filename=package://botdylan/meshes/components/f_knuckle/f_knuckle_E3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 scale=0.001 0.001 0.001
- link rh_rfmiddle: geometry collision cylinder length=0.025 radius=0.007; collision sphere radius=0.007
- link rh_rfproximal: geometry collision cylinder length=0.040 radius=0.007; visual mesh filename=package://botdylan/meshes/components/f_proximal/f_proximal_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 scale=0.001 0.001 0.001
- link rh_thdistal: geometry collision mesh filename=package://botdylan/meshes/components/th_distal/pst/th_dista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 scale=0.001 0.001 0.001; visual mesh filename=package://botdylan/meshes/components/th_distal/pst/th_dista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 scale=0.001 0.001 0.001
- link rh_thmiddle: geometry collision cylinder length=0.018 radius=0.011; collision sphere radius=0.011
- link rh_thproximal: geometry collision cylinder length=0.018 radius=0.012; visual mesh filename=package://botdylan/meshes/components/th_proximal/th_proxima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 scale=0.001 0.001 0.001
- link rh_wrist: geometry collision box size=0.027 0.018 0.010; collision box size=0.027 0.018 0.010
