Commit message: m

File: hand/xacro/finger/distal/distal.urdf.xacro (robot description, xacro)
@@ -44,13 +44,13 @@
         <geometry name="${prefix}${link_prefix}distal_visual">
           <xacro:if value="${tip_sensor == 'pst'}">
-            <mesh filename="package://sr_description/meshes/components/f_distal/pst/f_distal_pst.dae"
+            <mesh filename="package://botdylan/meshes/components/f_distal/pst/f_distal_pst.dae"
                   scale="0.001 0.001 0.001" />
           </xacro:if>
           <xacro:if value="${tip_sensor == 'bt_sp'}">
-            <mesh filename="package://sr_description/meshes/components/f_distal/bt_sp/f_distal_bt_sp.dae"
+            <mesh filename="package://botdylan/meshes/components/f_distal/bt_sp/f_distal_bt_sp.dae"
                   scale="0.001 0.001 0.001" />
           </xacro:if>
           <xacro:if value="${tip_sensor == 'bt_2p'}">
-            <mesh filename="package://sr_description/meshes/components/f_distal/bt_2p/f_distal_bt_2p.dae" />
+            <mesh filename="package://botdylan/meshes/components/f_distal/bt_2p/f_distal_bt_2p.dae" />
           </xacro:if>
         </geometry>
@@ -60,13 +60,13 @@
         <geometry name="${prefix}${link_prefix}distal_collision_geom">
           <xacro:if value="${tip_sensor == 'pst'}">
-            <mesh filename="package://sr_description/meshes/components/f_distal/pst/f_distal_pst.dae"
+            <mesh filename="package://botdylan/meshes/components/f_distal/pst/f_distal_pst.dae"
                   scale="0.001 0.001 0.001" />
           </xacro:if>
           <xacro:if value="${tip_sensor == 'bt_sp'}">
-            <mesh filename="package://sr_description/meshes/components/f_distal/bt_sp/f_distal_bt_sp.dae"
+            <mesh filename="package://botdylan/meshes/components/f_distal/bt_sp/f_distal_bt_sp.dae"
                   scale="0.001 0.001 0.001" />
           </xacro:if>
           <xacro:if value="${tip_sensor == 'bt_2p'}">
-            <mesh filename="package://sr_description/meshes/components/f_distal/bt_2p/f_distal_bt_2p.dae" />
+            <mesh filename="package://botdylan/meshes/components/f_distal/bt_2p/f_distal_bt_2p.dae" />
           </xacro:if>
         </geometry>

File: hand/xacro/finger/knuckle/knuckle.urdf.xacro (robot description, xacro)
@@ -43,5 +43,5 @@
         <origin xyz="0 0 0.0005" rpy="0 0 0" />
         <geometry name="${prefix}${link_prefix}knuckle_visual">
-          <mesh filename="package://sr_description/meshes/components/f_knuckle/f_knuckle_${hand_version}.dae" scale="0.001 0.001 0.001" />
+          <mesh filename="package://botdylan/meshes/components/f_knuckle/f_knuckle_${hand_version}.dae" scale="0.001 0.001 0.001" />
         </geometry>
         <material name="LightGrey" />

File: hand/xacro/thumb/thdistal.urdf.xacro (robot description, xacro)
@@ -65,5 +65,5 @@
           <origin xyz="0 0 0" rpy="0 0 0" />
           <geometry name="${prefix}th_distal_visual">
-            <mesh filename="package://sr_description/meshes/components/th_distal/bt_2p/th_distal_bt_2p.dae"
+            <mesh filename="package://botdylan/meshes/components/th_distal/bt_2p/th_distal_bt_2p.dae"
             scale="0.0254 0.0254 0.0254" />
           </geometry>
@@ -72,5 +72,5 @@
         <collision>
           <geometry name="${prefix}th_distal_collision_geom">
-            <mesh filename="package://sr_description/meshes/components/th_distal/bt_2p/th_distal_bt_2p.dae"
+            <mesh filename="package://botdylan/meshes/components/th_distal/bt_2p/th_distal_bt_2p.dae"
             scale="0.0254 0.0254 0.0254" />
           </geometry>
@@ -130,13 +130,13 @@
           <geometry name="${prefix}thdistal_visual">
             <xacro:if value="${tip_sensor == 'pst'}">
-              <mesh filename="package://sr_description/meshes/components/th_distal/pst/th_distal_pst.dae"
+              <mesh filename="package://botdylan/meshes/components/th_distal/pst/th_distal_pst.dae"
                     scale="0.001 0.001 0.001" />
             </xacro:if>
             <xacro:if value="${tip_sensor == 'bt_sp'}">
-              <mesh filename="package://sr_description/meshes/components/th_distal/bt_sp/th_distal_bt_sp.dae"
+              <mesh filename="package://botdylan/meshes/components/th_distal/bt_sp/th_distal_bt_sp.dae"
                     scale="0.001 0.001 0.001" />
             </xacro:if>
             <xacro:if value="${tip_sensor == 'bt_2p'}">
-              <mesh filename="package://sr_description/meshes/components/th_distal/bt_2p/th_distal_bt_2p.dae"
+              <mesh filename="package://botdylan/meshes/components/th_distal/bt_2p/th_distal_bt_2p.dae"
                     scale="0.001 0.001 0.001" />
             </xacro:if>
@@ -150,13 +150,13 @@
           <geometry name="${prefix}thmiddle_collision_geom">
             <xacro:if value="${tip_sensor == 'pst'}">
-              <mesh filename="package://sr_description/meshes/components/th_distal/pst/th_distal_pst.dae"
+              <mesh filename="package://botdylan/meshes/components/th_distal/pst/th_distal_pst.dae"
                     scale="0.001 0.001 0.001" />
             </xacro:if>
             <xacro:if value="${tip_sensor == 'bt_sp'}">
-              <mesh filename="package://sr_description/meshes/components/th_distal/bt_sp/th_distal_bt_sp.dae"
+              <mesh filename="package://botdylan/meshes/components/th_distal/bt_sp/th_distal_bt_sp.dae"
                     scale="0.001 0.001 0.001" />
             </xacro:if>
             <xacro:if value="${tip_sensor == 'bt_2p'}">
-              <mesh filename="package://sr_description/meshes/components/th_distal/bt_2p/th_distal_bt_2p.dae"
+              <mesh filename="package://botdylan/meshes/components/th_distal/bt_2p/th_distal_bt_2p.dae"
                     scale="0.001 0.001 0.001" />
             </xacro:if>

File: hand/xacro/thumb/thmiddle.urdf.xacro (robot description, xacro)
@@ -45,5 +45,5 @@
         <xacro:if value="${mid_sensor == 'bt_2p'}">
           <geometry name="${prefix}thmiddle_visual">
-            <mesh filename="package://sr_description/meshes/components/th_distal/bt_2p/th_distal_bt_2p_adapter.dae"
+            <mesh filename="package://botdylan/meshes/components/th_distal/bt_2p/th_distal_bt_2p_adapter.dae"
             scale="0.001 0.001 0.001" />
           </geometry>
@@ -51,5 +51,5 @@
         <xacro:unless value="${mid_sensor == 'bt_2p'}">
           <geometry name="${prefix}thmiddle_visual">
-            <mesh filename="package://sr_description/meshes/components/th_middle/th_middle_${hand_version}.dae"
+            <mesh filename="package://botdylan/meshes/components/th_middle/th_middle_${hand_version}.dae"
             scale="0.001 0.001 0.001" />
           </geometry>

File: urdf/sr_hand_bimanual.urdf (robot description, URDF)
Before this commit: robot bimanual_shadowhand_motor, 65 links, 64 joints
Links:
- link rh_palm: geometry collision box size=0.018 0.024 0.004; collision box size=0.020 0.024 0.040
- link rh_wrist: geometry collision box size=0.027 0.018 0.010; collision box size=0.027 0.018 0.010
