Commit message: Changes

File: hand/xacro/finger/lfmetacarpal/lfmetacarpal.urdf.xacro (robot description, xacro)
@@ -44,5 +44,5 @@
         <axis xyz="0.573576436 0 ${reflect*0.819152044}" />
         <geometry name="${prefix}lfmetacarpal_visual">
-          <mesh filename="package://sr_description/meshes/components/lf_metacarpal/lf_metacarpal_${hand_version}.dae"
+          <mesh filename="package://botdylan/meshes/components/lf_metacarpal/lf_metacarpal_${hand_version}.dae"
           scale="${reflect*0.001} 0.001 0.001" />
         </geometry>

File: hand/xacro/finger/middle/middle.urdf.xacro (robot description, xacro)
@@ -43,5 +43,5 @@
         <origin xyz="0 0 0" rpy="0 0 0" />
         <geometry name="${prefix}${link_prefix}middle_visual">
-          <mesh filename="package://sr_description/meshes/components/f_middle/f_middle_${hand_version}.dae"
+          <mesh filename="package://botdylan/meshes/components/f_middle/f_middle_${hand_version}.dae"
                 scale="0.001 0.001 0.001" />
         </geometry>

File: hand/xacro/finger/middle/middle_and_distal_bt_2p.urdf.xacro (robot description, xacro)
@@ -42,5 +42,5 @@
         <origin xyz="0 0 0" rpy="0 0 1.571" />
         <geometry name="${prefix}${link_prefix}middle_visual">
-          <mesh filename="package://sr_description/meshes/components/f_distal/bt_2p/f_distal_bt_2p_adapter.dae" />
+          <mesh filename="package://botdylan/meshes/components/f_distal/bt_2p/f_distal_bt_2p_adapter.dae" />
         </geometry>
         <material name="LightGrey" />
@@ -113,5 +113,5 @@
         <origin xyz="0 0 0" rpy="0 0 0" />
         <geometry name="${prefix}${link_prefix}distal_visual">
-          <mesh filename="package://sr_description/meshes/components/f_distal/bt_2p/f_distal_bt_2p.dae"
+          <mesh filename="package://botdylan/meshes/components/f_distal/bt_2p/f_distal_bt_2p.dae"
                 scale="0.0254 0.0254 0.0254" />
         </geometry>
@@ -119,5 +119,5 @@
       <collision>
         <geometry name="${prefix}${link_prefix}distal_collision_geom">
-          <mesh filename="package://sr_description/meshes/components/f_distal/bt_2p/f_distal_bt_2p.dae"
+          <mesh filename="package://botdylan/meshes/components/f_distal/bt_2p/f_distal_bt_2p.dae"
                 scale="0.0254 0.0254 0.0254" />
         </geometry>

File: hand/xacro/finger/proximal/proximal.urdf.xacro (robot description, xacro)
@@ -43,5 +43,5 @@
         <origin xyz="0 0 0" rpy="0 0 0" />
         <geometry name="${prefix}${link_prefix}proximal_visual">
-          <mesh filename="package://sr_description/meshes/components/f_proximal/f_proximal_${hand_version}.dae"
+          <mesh filename="package://botdylan/meshes/components/f_proximal/f_proximal_${hand_version}.dae"
                 scale="0.001 0.001 0.001" />
         </geometry>

File: hand/xacro/forearm/forearm_c.urdf.xacro (robot description, xacro)
@@ -45,5 +45,5 @@
         <origin xyz="0 0 0" rpy="0 0 0" />
         <geometry name="${prefix}forearm_visual">
-          <mesh filename="package://sr_description/meshes/components/forearm/forearm_${hand_version}.dae"/>
+          <mesh filename="package://botdylan/meshes/components/forearm/forearm_${hand_version}.dae"/>
         </geometry>
         <material name="Grey" />

File: hand/xacro/forearm/forearm_e.urdf.xacro (robot description, xacro)
@@ -51,5 +51,5 @@
         <origin xyz="0 0 ${mounting_plate_offset}" rpy="0 0 0" />
         <geometry name="${prefix}forearm_visual">
-          <mesh filename="package://sr_description/meshes/components/forearm/forearm_${hand_version}.dae" scale="0.001 0.001 0.001" />
+          <mesh filename="package://botdylan/meshes/components/forearm/forearm_${hand_version}.dae" scale="0.001 0.001 0.001" />
         </geometry>
         <xacro:light_grey/>
@@ -58,5 +58,5 @@
         <origin xyz="0 0 ${mounting_plate_offset}" rpy="0 0 0" />
         <geometry name="${prefix}forearm_collision">
-          <mesh filename="package://sr_description/meshes/components/forearm/forearm_collision_${hand_version}.dae" scale="0.001 0.001 0.001" />
+          <mesh filename="package://botdylan/meshes/components/forearm/forearm_collision_${hand_version}.dae" scale="0.001 0.001 0.001" />
         </geometry>
       </collision>
@@ -73,5 +73,5 @@
           <origin xyz="0 0 0" rpy="0 0 0" />
           <geometry name="${prefix}mounting_plate">
-            <mesh filename="package://sr_description/meshes/components/mounting_plate/mounting_plate_${hand_version}.dae" scale="0.001 0.001 0.001" />
+            <mesh filename="package://botdylan/meshes/components/mounting_plate/mounting_plate_${hand_version}.dae" scale="0.001 0.001 0.001" />
           </geometry>
         </visual>

File: hand/xacro/forearm/forearm_g.urdf.xacro (robot description, xacro)
@@ -42,5 +42,5 @@
         <origin xyz="0 0 ${mounting_plate_offset}" rpy="0 0 ${pi/2}" />
         <geometry name="${prefix}forearm_visual">
-          <mesh filename="package://sr_description/meshes/components/forearm/forearm_${hand_version}.dae" scale="1.0 1.0 1.0" />
+          <mesh filename="package://botdylan/meshes/components/forearm/forearm_${hand_version}.dae" scale="1.0 1.0 1.0" />
         </geometry>
         <material name="Grey" />
@@ -57,5 +57,5 @@
           <origin xyz="0 0 0" rpy="0 0 0" />
           <geometry name="${prefix}mounting_plate">
-            <mesh filename="package://sr_description/meshes/components/mounting_plate/mounting_plate_${hand_version}.dae" scale="0.001 0.001 0.001" />
+            <mesh filename="package://botdylan/meshes/components/mounting_plate/mounting_plate_${hand_version}.dae" scale="0.001 0.001 0.001" />
           </geometry>
         </visual>

File: hand/xacro/palm/palm_e.urdf.xacro (robot description, xacro)
@@ -44,5 +44,5 @@
         <origin xyz="0 0 0" rpy="0 0 0" />
         <geometry name="${prefix}palm_visual">
-          <mesh filename="package://sr_description/meshes/components/palm/palm_${hand_version}.dae"
+          <mesh filename="package://botdylan/meshes/components/palm/palm_${hand_version}.dae"
                 scale="${reflect*0.001} 0.001 0.001" />
         </geometry>

File: hand/xacro/palm/palm_g.urdf.xacro (robot description, xacro)
@@ -43,5 +43,5 @@
         <origin xyz="0 0 0" rpy="0 0 0" />
         <geometry name="${prefix}palm_visual">
-          <mesh filename="package://sr_description/meshes/components/palm/palm_${hand_version}.dae"
+          <mesh filename="package://botdylan/meshes/components/palm/palm_${hand_version}.dae"
           scale="${reflect*0.001} 0.001 0.001" />
         </geometry>

File: hand/xacro/thumb/thproximal.urdf.xacro (robot description, xacro)
@@ -43,5 +43,5 @@
         <origin xyz="0 0 0" rpy="0 0 0" />
         <geometry name="${prefix}thproximal_visual">
-          <mesh filename="package://sr_description/meshes/components/th_proximal/th_proximal_${hand_version}.dae"
+          <mesh filename="package://botdylan/meshes/components/th_proximal/th_proximal_${hand_version}.dae"
           scale="0.001 0.001 0.001" />
         </geometry>

File: urdf/sr_hand_bimanual.urdf (robot description, URDF)
Before this commit: robot bimanual_shadowhand_motor, 65 links, 64 joints
Links:
- link rh_palm: geometry collision box size=0.018 0.024 0.004; collision box size=0.020 0.024 0.040
- link rh_wrist: geometry collision box size=0.027 0.018 0.010; collision box size=0.027 0.018 0.010
