Commit message: m

File: urdf/sr_hand_bimanual.urdf (robot description, URDF)
Before this commit: robot bimanual_shadowhand_motor, 65 links, 64 joints
Links:
- added link guitar-neck; collision box size=0.02 0.60 0.30; visual box size=0.02 0.60 0.30
Joints:
- added joint attach-guitar-neck: type fixed, parent world, child guitar, origin xyz=0.00 1.0 0 rpy=0 0 0

Commit message: m

File: urdf/sr_hand_bimanual.urdf (robot description, URDF)
Before this commit: robot bimanual_shadowhand_motor, 66 links, 65 joints
Links:
- removed link guitar-neck
- added link neck, mass 0.5; collision box size=0.8 0.05 0.02; visual box size=0.8 0.05 0.02
- added link string_1, mass 0.01; collision cylinder length=0.8 radius=0.001; visual cylinder length=0.8 radius=0.001
- added link string_2, mass 0.01; collision cylinder length=0.8 radius=0.001; visual cylinder length=0.8 radius=0.001
- added link string_3, mass 0.01; collision cylinder length=0.8 radius=0.001; visual cylinder length=0.8 radius=0.001
- added link string_4, mass 0.01; collision cylinder length=0.8 radius=0.001; visual cylinder length=0.8 radius=0.001
- added link string_5, mass 0.01; collision cylinder length=0.8 radius=0.001; visual cylinder length=0.8 radius=0.001
- added link string_6, mass 0.01; collision cylinder length=0.8 radius=0.001; visual cylinder length=0.8 radius=0.001
Joints:
- removed joint attach-guitar-neck
- added joint string_1_to_neck: type fixed, parent neck, child string_1, origin xyz=0 -0.02 0.01 rpy=0 0 0
- added joint string_2_to_neck: type fixed, parent neck, child string_2, origin xyz=0 -0.012 0.01 rpy=0 0 0
- added joint string_3_to_neck: type fixed, parent neck, child string_3, origin xyz=0 -0.004 0.01 rpy=0 0 0
- added joint string_4_to_neck: type fixed, parent neck, child string_4, origin xyz=0 0.004 0.01 rpy=0 0 0
- added joint string_5_to_neck: type fixed, parent neck, child string_5, origin xyz=0 0.012 0.01 rpy=0 0 0
- added joint string_6_to_neck: type fixed, parent neck, child string_6, origin xyz=0 0.02 0.01 rpy=0 0 0

Commit message: m

File: urdf/sr_hand_bimanual.urdf (robot description, URDF)
Before this commit: robot bimanual_shadowhand_motor, 65 links, 64 joints
Links:
- link lh_ffdistal: geometry collision mesh filename=package://meshes/components/f_distal/pst/f_distal_pst.dae scale=0.001 0.001 0.001; visual mesh filename=package://meshes/components/f_distal/pst/f_distal_pst.dae scale=0.001 0.001 0.001
- link lh_ffknuckle: geometry collision cylinder length=0.014 radius=0.007; visual mesh filename=package://meshes/components/f_knuckle/f_knuckle_E3M5.dae scale=0.001 0.001 0.001
- link lh_ffmiddle: geometry collision cylinder length=0.025 radius=0.007; collision sphere radius=0.007
- link lh_ffproximal: geometry collision cylinder length=0.040 radius=0.007; visual mesh filename=package://meshes/components/f_proximal/f_proximal_E3M5.dae scale=0.001 0.001 0.001
- link lh_forearm: geometry collision box size=0.07 0.07 0.07; collision mesh filename=package://meshes/components/forearm/forearm_collision_E3M5.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 scale=0.001 0.001 0.001
- link lh_lfdistal: geometry collision mesh filename=package://meshes/components/f_distal/pst/f_distal_pst.dae scale=0.001 0.001 0.001; visual mesh filename=package://meshes/components/f_distal/pst/f_distal_pst.dae scale=0.001 0.001 0.001
- link lh_lfknuckle: geometry collision cylinder length=0.014 radius=0.007; visual mesh filename=package://meshes/components/f_knuckle/f_knuckle_E3M5.dae scale=0.001 0.001 0.001
- link lh_lfmetacarpal: geometry collision box size=0.018 0.024 0.040; visual mesh filename=package://meshes/components/lf_metacarpal/lf_metacarpal_E3M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 scale=-0.001 0.001 0.001
- link lh_lfmiddle: geometry collision cylinder length=0.025 radius=0.007; collision sphere radius=0.007
- link lh_lfproximal: geometry collision cylinder length=0.040 radius=0.007; visual mesh filename=package://meshes/components/f_proximal/f_proximal_E3M5.dae scale=0.001 0.001 0.001
- link lh_mfdistal: geometry collision mesh filename=package://meshes/components/f_distal/pst/f_distal_pst.dae scale=0.001 0.001 0.001; visual mesh filename=package://meshes/components/f_distal/pst/f_distal_pst.dae scale=0.001 0.001 0.001
- link lh_mfknuckle: geometry collision cylinder length=0.014 radius=0.007; visual mesh filename=package://meshes/components/f_knuckle/f_knuckle_E3M5.dae scale=0.001 0.001 0.001
- link lh_mfmiddle: geometry collision cylinder length=0.025 radius=0.007; collision sphere radius=0.007
- link lh_mfproximal: geometry collision cylinder length=0.040 radius=0.007; visual mesh filename=package://meshes/components/f_proximal/f_proximal_E3M5.dae scale=0.001 0.001 0.001
- link lh_palm: geometry collision box size=0.018 0.024 0.004; collision box size=0.020 0.024 0.040
- link lh_rfdistal: geometry collision mesh filename=package://meshes/components/f_distal/pst/f_distal_pst.dae scale=0.001 0.001 0.001; visual mesh filename=package://meshes/components/f_distal/pst/f_distal_pst.dae scale=0.001 0.001 0.001
- link lh_rfknuckle: geometry collision cylinder length=0.014 radius=0.007; visual mesh filename=package://meshes/components/f_knuckle/f_knuckle_E3M5.dae scale=0.001 0.001 0.001
- link lh_rfmiddle: geometry collision cylinder length=0.025 radius=0.007; collision sphere radius=0.007
- link lh_rfproximal: geometry collision cylinder length=0.040 radius=0.007; visual mesh filename=package://meshes/components/f_proximal/f_proximal_E3M5.dae scale=0.001 0.001 0.001
- link lh_thdistal: geometry collision mesh filename=package://meshes/components/th_distal/pst/th_distal_pst.dae scale=0.001 0.001 0.001; visual mesh filename=package://meshes/components/th_distal/pst/th_distal_pst.dae scale=0.001 0.001 0.001
- link lh_thmiddle: geometry collision cylinder length=0.018 radius=0.011; collision sphere radius=0.011
- link lh_thproximal: geometry collision cylinder length=0.018 radius=0.012; visual mesh filename=package://meshes/components/th_proximal/th_proximal_E3M5.dae scale=0.001 0.001 0.001
- link lh_wrist: geometry collision box size=0.027 0.018 0.010; collision box size=0.027 0.018 0.010
- link rh_ffdistal: geometry collision mesh filename=package://meshes/components/f_distal/pst/f_distal_pst.dae scale=0.001 0.001 0.001; visual mesh filename=package://meshes/components/f_distal/pst/f_distal_pst.dae scale=0.001 0.001 0.001
- link rh_ffknuckle: geometry collision cylinder length=0.014 radius=0.007; visual mesh filename=package://meshes/components/f_knuckle/f_knuckle_E3M5.dae scale=0.001 0.001 0.001
- link rh_ffmiddle: geometry collision cylinder length=0.025 radius=0.007; collision sphere radius=0.007
- link rh_ffproximal: geometry collision cylinder length=0.040 radius=0.007; visual mesh filename=package://meshes/components/f_proximal/f_proximal_E3M5.dae scale=0.001 0.001 0.001
- link rh_forearm: geometry collision box size=0.07 0.07 0.07; collision mesh filename=package://meshes/components/forearm/forearm_collision_E3M5.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 scale=0.001 0.001 0.001
- link rh_lfdistal: geometry collision mesh filename=package://meshes/components/f_distal/pst/f_distal_pst.dae scale=0.001 0.001 0.001; visual mesh filename=package://meshes/components/f_distal/pst/f_distal_pst.dae scale=0.001 0.001 0.001
- link rh_lfknuckle: geometry collision cylinder length=0.014 radius=0.007; visual mesh filename=package://meshes/components/f_knuckle/f_knuckle_E3M5.dae scale=0.001 0.001 0.001
- link rh_lfmetacarpal: geometry collision box size=0.018 0.024 0.040; visual mesh filename=package://meshes/components/lf_metacarpal/lf_metacarpal_E3M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 scale=0.001 0.001 0.001
- link rh_lfmiddle: geometry collision cylinder length=0.025 radius=0.007; collision sphere radius=0.007
- link rh_lfproximal: geometry collision cylinder length=0.040 radius=0.007; visual mesh filename=package://meshes/components/f_proximal/f_proximal_E3M5.dae scale=0.001 0.001 0.001
- link rh_mfdistal: geometry collision mesh filename=package://meshes/components/f_distal/pst/f_distal_pst.dae scale=0.001 0.001 0.001; visual mesh filename=package://meshes/components/f_distal/pst/f_distal_pst.dae scale=0.001 0.001 0.001
- link rh_mfknuckle: geometry collision cylinder length=0.014 radius=0.007; visual mesh filename=package://meshes/components/f_knuckle/f_knuckle_E3M5.dae scale=0.001 0.001 0.001
- link rh_mfmiddle: geometry collision cylinder length=0.025 radius=0.007; collision sphere radius=0.007
- link rh_mfproximal: geometry collision cylinder length=0.040 radius=0.007; visual mesh filename=package://meshes/components/f_proximal/f_proximal_E3M5.dae scale=0.001 0.001 0.001
- link rh_palm: geometry collision box size=0.018 0.024 0.004; collision box size=0.020 0.024 0.040
- link rh_rfdistal: geometry collision mesh filename=package://meshes/components/f_distal/pst/f_distal_pst.dae scale=0.001 0.001 0.001; visual mesh filename=package://meshes/components/f_distal/pst/f_distal_pst.dae scale=0.001 0.001 0.001
- link rh_rfknuckle: geometry collision cylinder length=0.014 radius=0.007; visual mesh filename=package://meshes/components/f_knuckle/f_knuckle_E3M5.dae scale=0.001 0.001 0.001
- link rh_rfmiddle: geometry collision cylinder length=0.025 radius=0.007; collision sphere radius=0.007
- link rh_rfproximal: geometry collision cylinder length=0.040 radius=0.007; visual mesh filename=package://meshes/components/f_proximal/f_proximal_E3M5.dae scale=0.001 0.001 0.001
- link rh_thdistal: geometry collision mesh filename=package://meshes/components/th_distal/pst/th_distal_pst.dae scale=0.001 0.001 0.001; visual mesh filename=package://meshes/components/th_distal/pst/th_distal_pst.dae scale=0.001 0.001 0.001
- link rh_thmiddle: geometry collision cylinder length=0.018 radius=0.011; collision sphere radius=0.011
- link rh_thproximal: geometry collision cylinder length=0.018 radius=0.012; visual mesh filename=package://meshes/components/th_proximal/th_proximal_E3M5.dae scale=0.001 0.001 0.001
- link rh_wrist: geometry collision box size=0.027 0.018 0.010; collision box size=0.027 0.018 0.010

Commit message: m

File: urdf/sr_hand_bimanual.urdf (robot description, URDF)
Before this commit: robot bimanual_shadowhand_motor, 65 links, 64 joints
Links:
- added link neck, mass 0.5; collision box size=0.8 0.05 0.02; visual box size=0.8 0.05 0.02
- added link string_1, mass 0.01; collision cylinder length=0.8 radius=0.001; visual cylinder length=0.8 radius=0.001
- added link string_2, mass 0.01; collision cylinder length=0.8 radius=0.001; visual cylinder length=0.8 radius=0.001
- added link string_3, mass 0.01; collision cylinder length=0.8 radius=0.001; visual cylinder length=0.8 radius=0.001
- added link string_4, mass 0.01; collision cylinder length=0.8 radius=0.001; visual cylinder length=0.8 radius=0.001
- added link string_5, mass 0.01; collision cylinder length=0.8 radius=0.001; visual cylinder length=0.8 radius=0.001
- added link string_6, mass 0.01; collision cylinder length=0.8 radius=0.001; visual cylinder length=0.8 radius=0.001
Joints:
- added joint neck_to_world: type None, parent world, child neck, origin xyz=0 0 0 rpy=0 0 0
- added joint string_1_to_neck: type fixed, parent neck, child string_1, origin xyz=0 -0.02 0.01 rpy=0 0 0
- added joint string_2_to_neck: type fixed, parent neck, child string_2, origin xyz=0 -0.012 0.01 rpy=0 0 0
- added joint string_3_to_neck: type fixed, parent neck, child string_3, origin xyz=0 -0.004 0.01 rpy=0 0 0
- added joint string_4_to_neck: type fixed, parent neck, child string_4, origin xyz=0 0.004 0.01 rpy=0 0 0
- added joint string_5_to_neck: type fixed, parent neck, child string_5, origin xyz=0 0.012 0.01 rpy=0 0 0
- added joint string_6_to_neck: type fixed, parent neck, child string_6, origin xyz=0 0.02 0.01 rpy=0 0 0

Commit message: m

File: urdf/sr_hand_bimanual.urdf (robot description, URDF)
Before this commit: robot bimanual_shadowhand_motor, 72 links, 71 joints
Joints:
- joint neck_to_world: type None -> fixed

Commit message: Pushing for fidelity

File: urdf/sr_hand_bimanual.urdf (robot description, URDF)
Before this commit: robot bimanual_shadowhand_motor, 72 links, 71 joints
Joints:
- removed joint neck_to_world
- added joint neck_to_lh_lftip: type fixed, parent lh_lftip, child neck, origin xyz=0 0 0 rpy=0 0 0

Commit message: Attach guitar to world

File: urdf/sr_hand_bimanual.urdf (robot description, URDF)
Before this commit: robot bimanual_shadowhand_motor, 72 links, 71 joints
Joints:
- removed joint neck_to_lh_lftip
- added joint neck_to_world: type fixed, parent world, child neck, origin xyz=0 0 0 rpy=0 0 0

Commit message: m

File: urdf/sr_hand_bimanual.urdf (robot description, URDF)
Before this commit: robot bimanual_shadowhand_motor, 72 links, 71 joints
Links:
- link lh_ffdistal: geometry collision mesh filename=package://botdylan/meshes/components/f_distal/pst/f_distal_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 scale=0.001 0.001 0.001; visual mesh filename=package://botdylan/meshes/components/f_distal/pst/f_distal_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 scale=0.001 0.001 0.001
- link lh_ffknuckle: geometry collision cylinder length=0.014 radius=0.007; visual mesh filename=package://botdylan/meshes/components/f_knuckle/f_knuckle_E3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 scale=0.001 0.001 0.001
- link lh_ffmiddle: geometry collision cylinder length=0.025 radius=0.007; collision sphere radius=0.007
- link lh_ffproximal: geometry collision cylinder length=0.040 radius=0.007; visual mesh filename=package://botdylan/meshes/components/f_proximal/f_proximal_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 scale=0.001 0.001 0.001
- link lh_forearm: geometry collision box size=0.07 0.07 0.07; collision mesh filename=package://botdylan/meshes/components/forearm/forearm_collis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 scale=0.001 0.001 0.001
- link lh_lfdistal: geometry collision mesh filename=package://botdylan/meshes/components/f_distal/pst/f_distal_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 scale=0.001 0.001 0.001; visual mesh filename=package://botdylan/meshes/components/f_distal/pst/f_distal_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 scale=0.001 0.001 0.001
- link lh_lfknuckle: geometry collision cylinder length=0.014 radius=0.007; visual mesh filename=package://botdylan/meshes/components/f_knuckle/f_knuckle_E3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 scale=0.001 0.001 0.001
- link lh_lfmetacarpal: geometry collision box size=0.018 0.024 0.040; visual mesh filename=package://botdylan/meshes/components/lf_metacarpal/lf_metac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 scale=-0.001 0.001 0.001
- link lh_lfmiddle: geometry collision cylinder length=0.025 radius=0.007; collision sphere radius=0.007
- link lh_lfproximal: geometry collision cylinder length=0.040 radius=0.007; visual mesh filename=package://botdylan/meshes/components/f_proximal/f_proximal_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 scale=0.001 0.001 0.001
- link lh_mfdistal: geometry collision mesh filename=package://botdylan/meshes/components/f_distal/pst/f_distal_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 scale=0.001 0.001 0.001; visual mesh filename=package://botdylan/meshes/components/f_distal/pst/f_distal_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 scale=0.001 0.001 0.001
- link lh_mfknuckle: geometry collision cylinder length=0.014 radius=0.007; visual mesh filename=package://botdylan/meshes/components/f_knuckle/f_knuckle_E3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 scale=0.001 0.001 0.001
- link lh_mfmiddle: geometry collision cylinder length=0.025 radius=0.007; collision sphere radius=0.007
- link lh_mfproximal: geometry collision cylinder length=0.040 radius=0.007; visual mesh filename=package://botdylan/meshes/components/f_proximal/f_proximal_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 scale=0.001 0.001 0.001
- link lh_palm: geometry collision box size=0.018 0.024 0.004; collision box size=0.020 0.024 0.040
- link lh_rfdistal: geometry collision mesh filename=package://botdylan/meshes/components/f_distal/pst/f_distal_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 scale=0.001 0.001 0.001; visual mesh filename=package://botdylan/meshes/components/f_distal/pst/f_distal_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 scale=0.001 0.001 0.001
- link lh_rfknuckle: geometry collision cylinder length=0.014 radius=0.007; visual mesh filename=package://botdylan/meshes/components/f_knuckle/f_knuckle_E3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 scale=0.001 0.001 0.001
- link lh_rfmiddle: geometry collision cylinder length=0.025 radius=0.007; collision sphere radius=0.007
- link lh_rfproximal: geometry collision cylinder length=0.040 radius=0.007; visual mesh filename=package://botdylan/meshes/components/f_proximal/f_proximal_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 scale=0.001 0.001 0.001
- link lh_thdistal: geometry collision mesh filename=package://botdylan/meshes/components/th_distal/pst/th_dista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 scale=0.001 0.001 0.001; visual mesh filename=package://botdylan/meshes/components/th_distal/pst/th_dista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 scale=0.001 0.001 0.001
- link lh_thmiddle: geometry collision cylinder length=0.018 radius=0.011; collision sphere radius=0.011
- link lh_thproximal: geometry collision cylinder length=0.018 radius=0.012; visual mesh filename=package://botdylan/meshes/components/th_proximal/th_proxima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 scale=0.001 0.001 0.001
- link lh_wrist: geometry collision box size=0.027 0.018 0.010; collision box size=0.027 0.018 0.010
- link rh_ffdistal: geometry collision mesh filename=package://botdylan/meshes/components/f_distal/pst/f_distal_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 scale=0.001 0.001 0.001; visual mesh filename=package://botdylan/meshes/components/f_distal/pst/f_distal_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 scale=0.001 0.001 0.001
- link rh_ffknuckle: geometry collision cylinder length=0.014 radius=0.007; visual mesh filename=package://botdylan/meshes/components/f_knuckle/f_knuckle_E3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 scale=0.001 0.001 0.001
- link rh_ffmiddle: geometry collision cylinder length=0.025 radius=0.007; collision sphere radius=0.007
- link rh_ffproximal: geometry collision cylinder length=0.040 radius=0.007; visual mesh filename=package://botdylan/meshes/components/f_proximal/f_proximal_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 scale=0.001 0.001 0.001
- link rh_forearm: geometry collision box size=0.07 0.07 0.07; collision mesh filename=package://botdylan/meshes/components/forearm/forearm_collis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 scale=0.001 0.001 0.001
- link rh_lfdistal: geometry collision mesh filename=package://botdylan/meshes/components/f_distal/pst/f_distal_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 scale=0.001 0.001 0.001; visual mesh filename=package://botdylan/meshes/components/f_distal/pst/f_distal_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 scale=0.001 0.001 0.001
- link rh_lfknuckle: geometry collision cylinder length=0.014 radius=0.007; visual mesh filename=package://botdylan/meshes/components/f_knuckle/f_knuckle_E3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 scale=0.001 0.001 0.001
- link rh_lfmetacarpal: geometry collision box size=0.018 0.024 0.040; visual mesh filename=package://botdylan/meshes/components/lf_metacarpal/lf_metac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 scale=0.001 0.001 0.001
- link rh_lfmiddle: geometry collision cylinder length=0.025 radius=0.007; collision sphere radius=0.007
- link rh_lfproximal: geometry collision cylinder length=0.040 radius=0.007; visual mesh filename=package://botdylan/meshes/components/f_proximal/f_proximal_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 scale=0.001 0.001 0.001
- link rh_mfdistal: geometry collision mesh filename=package://botdylan/meshes/components/f_distal/pst/f_distal_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 scale=0.001 0.001 0.001; visual mesh filename=package://botdylan/meshes/components/f_distal/pst/f_distal_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 scale=0.001 0.001 0.001
- link rh_mfknuckle: geometry collision cylinder length=0.014 radius=0.007; visual mesh filename=package://botdylan/meshes/components/f_knuckle/f_knuckle_E3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 scale=0.001 0.001 0.001
- link rh_mfmiddle: geometry collision cylinder length=0.025 radius=0.007; collision sphere radius=0.007
- link rh_mfproximal: geometry collision cylinder length=0.040 radius=0.007; visual mesh filename=package://botdylan/meshes/components/f_proximal/f_proximal_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 scale=0.001 0.001 0.001
- link rh_palm: geometry collision box size=0.018 0.024 0.004; collision box size=0.020 0.024 0.040
- link rh_rfdistal: geometry collision mesh filename=package://botdylan/meshes/components/f_distal/pst/f_distal_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 scale=0.001 0.001 0.001; visual mesh filename=package://botdylan/meshes/components/f_distal/pst/f_distal_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 scale=0.001 0.001 0.001
- link rh_rfknuckle: geometry collision cylinder length=0.014 radius=0.007; visual mesh filename=package://botdylan/meshes/components/f_knuckle/f_knuckle_E3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 scale=0.001 0.001 0.001
- link rh_rfmiddle: geometry collision cylinder length=0.025 radius=0.007; collision sphere radius=0.007
- link rh_rfproximal: geometry collision cylinder length=0.040 radius=0.007; visual mesh filename=package://botdylan/meshes/components/f_proximal/f_proximal_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 scale=0.001 0.001 0.001
- link rh_thdistal: geometry collision mesh filename=package://botdylan/meshes/components/th_distal/pst/th_dista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 scale=0.001 0.001 0.001; visual mesh filename=package://botdylan/meshes/components/th_distal/pst/th_dista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 scale=0.001 0.001 0.001
- link rh_thmiddle: geometry collision cylinder length=0.018 radius=0.011; collision sphere radius=0.011
- link rh_thproximal: geometry collision cylinder length=0.018 radius=0.012; visual mesh filename=package://botdylan/meshes/components/th_proximal/th_proxima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 scale=0.001 0.001 0.001
- link rh_wrist: geometry collision box size=0.027 0.018 0.010; collision box size=0.027 0.018 0.010
