Commit message: m

File: urdf/sr_hand_bimanual.urdf (robot description, URDF)
Before this commit: robot bimanual_shadowhand_motor, 65 links, 64 joints
Links:
- link lh_ffdistal: geometry collision mesh filename=package://sr_description/meshes/components/f_distal/pst/f_d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 scale=0.001 0.001 0.001; visual mesh filename=package://sr_description/meshes/components/f_distal/pst/f_d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 scale=0.001 0.001 0.001
- link lh_ffknuckle: geometry collision cylinder length=0.014 radius=0.007; visual mesh filename=package://sr_description/meshes/components/f_knuckle/f_knuc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 scale=0.001 0.001 0.001
- link lh_ffmiddle: geometry collision cylinder length=0.025 radius=0.007; collision sphere radius=0.007
- link lh_ffproximal: geometry collision cylinder length=0.040 radius=0.007; visual mesh filename=package://sr_description/meshes/components/f_proximal/f_pro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 scale=0.001 0.001 0.001
- link lh_forearm: geometry collision box size=0.07 0.07 0.07; collision mesh filename=package://sr_description/meshes/components/forearm/forearm_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 scale=0.001 0.001 0.001
- link lh_lfdistal: geometry collision mesh filename=package://sr_description/meshes/components/f_distal/pst/f_d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 scale=0.001 0.001 0.001; visual mesh filename=package://sr_description/meshes/components/f_distal/pst/f_d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 scale=0.001 0.001 0.001
- link lh_lfknuckle: geometry collision cylinder length=0.014 radius=0.007; visual mesh filename=package://sr_description/meshes/components/f_knuckle/f_knuc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 scale=0.001 0.001 0.001
- link lh_lfmetacarpal: geometry collision box size=0.018 0.024 0.040; visual mesh filename=package://sr_description/meshes/components/lf_metacarpal/lf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 scale=-0.001 0.001 0.001
- link lh_lfmiddle: geometry collision cylinder length=0.025 radius=0.007; collision sphere radius=0.007
- link lh_lfproximal: geometry collision cylinder length=0.040 radius=0.007; visual mesh filename=package://sr_description/meshes/components/f_proximal/f_pro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 scale=0.001 0.001 0.001
- link lh_mfdistal: geometry collision mesh filename=package://sr_description/meshes/components/f_distal/pst/f_d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 scale=0.001 0.001 0.001; visual mesh filename=package://sr_description/meshes/components/f_distal/pst/f_d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 scale=0.001 0.001 0.001
- link lh_mfknuckle: geometry collision cylinder length=0.014 radius=0.007; visual mesh filename=package://sr_description/meshes/components/f_knuckle/f_knuc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 scale=0.001 0.001 0.001
- link lh_mfmiddle: geometry collision cylinder length=0.025 radius=0.007; collision sphere radius=0.007
- link lh_mfproximal: geometry collision cylinder length=0.040 radius=0.007; visual mesh filename=package://sr_description/meshes/components/f_proximal/f_pro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 scale=0.001 0.001 0.001
- link lh_palm: geometry collision box size=0.018 0.024 0.004; collision box size=0.020 0.024 0.040
- link lh_rfdistal: geometry collision mesh filename=package://sr_description/meshes/components/f_distal/pst/f_d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 scale=0.001 0.001 0.001; visual mesh filename=package://sr_description/meshes/components/f_distal/pst/f_d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 scale=0.001 0.001 0.001
- link lh_rfknuckle: geometry collision cylinder length=0.014 radius=0.007; visual mesh filename=package://sr_description/meshes/components/f_knuckle/f_knuc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 scale=0.001 0.001 0.001
- link lh_rfmiddle: geometry collision cylinder length=0.025 radius=0.007; collision sphere radius=0.007
- link lh_rfproximal: geometry collision cylinder length=0.040 radius=0.007; visual mesh filename=package://sr_description/meshes/components/f_proximal/f_pro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 scale=0.001 0.001 0.001
- link lh_thdistal: geometry collision mesh filename=package://sr_description/meshes/components/th_distal/pst/th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 scale=0.001 0.001 0.001; visual mesh filename=package://sr_description/meshes/components/th_distal/pst/th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 scale=0.001 0.001 0.001
- link lh_thmiddle: geometry collision cylinder length=0.018 radius=0.011; collision sphere radius=0.011
- link lh_thproximal: geometry collision cylinder length=0.018 radius=0.012; visual mesh filename=package://sr_description/meshes/components/th_proximal/th_p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 scale=0.001 0.001 0.001
- link lh_wrist: mass None -> 0.1; geometry collision box size=0.027 0.018 0.010; collision box size=0.027 0.018 0.010
- link rh_ffdistal: geometry collision mesh filename=package://sr_description/meshes/components/f_distal/pst/f_d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 scale=0.001 0.001 0.001; visual mesh filename=package://sr_description/meshes/components/f_distal/pst/f_d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 scale=0.001 0.001 0.001
- link rh_ffknuckle: geometry collision cylinder length=0.014 radius=0.007; visual mesh filename=package://sr_description/meshes/components/f_knuckle/f_knuc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 scale=0.001 0.001 0.001
- link rh_ffmiddle: geometry collision cylinder length=0.025 radius=0.007; collision sphere radius=0.007
- link rh_ffproximal: geometry collision cylinder length=0.040 radius=0.007; visual mesh filename=package://sr_description/meshes/components/f_proximal/f_pro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 scale=0.001 0.001 0.001
- link rh_forearm: geometry collision box size=0.07 0.07 0.07; collision mesh filename=package://sr_description/meshes/components/forearm/forearm_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 scale=0.001 0.001 0.001
- link rh_lfdistal: geometry collision mesh filename=package://sr_description/meshes/components/f_distal/pst/f_d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 scale=0.001 0.001 0.001; visual mesh filename=package://sr_description/meshes/components/f_distal/pst/f_d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 scale=0.001 0.001 0.001
- link rh_lfknuckle: geometry collision cylinder length=0.014 radius=0.007; visual mesh filename=package://sr_description/meshes/components/f_knuckle/f_knuc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 scale=0.001 0.001 0.001
- link rh_lfmetacarpal: geometry collision box size=0.018 0.024 0.040; visual mesh filename=package://sr_description/meshes/components/lf_metacarpal/lf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 scale=0.001 0.001 0.001
- link rh_lfmiddle: geometry collision cylinder length=0.025 radius=0.007; collision sphere radius=0.007
- link rh_lfproximal: geometry collision cylinder length=0.040 radius=0.007; visual mesh filename=package://sr_description/meshes/components/f_proximal/f_pro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 scale=0.001 0.001 0.001
- link rh_mfdistal: geometry collision mesh filename=package://sr_description/meshes/components/f_distal/pst/f_d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 scale=0.001 0.001 0.001; visual mesh filename=package://sr_description/meshes/components/f_distal/pst/f_d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 scale=0.001 0.001 0.001
- link rh_mfknuckle: geometry collision cylinder length=0.014 radius=0.007; visual mesh filename=package://sr_description/meshes/components/f_knuckle/f_knuc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 scale=0.001 0.001 0.001
- link rh_mfmiddle: geometry collision cylinder length=0.025 radius=0.007; collision sphere radius=0.007
- link rh_mfproximal: geometry collision cylinder length=0.040 radius=0.007; visual mesh filename=package://sr_description/meshes/components/f_proximal/f_pro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 scale=0.001 0.001 0.001
- link rh_palm: mass None -> 0.3; geometry collision box size=0.018 0.024 0.004; collision box size=0.020 0.024 0.040
- link rh_rfdistal: geometry collision mesh filename=package://sr_description/meshes/components/f_distal/pst/f_d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 scale=0.001 0.001 0.001; visual mesh filename=package://sr_description/meshes/components/f_distal/pst/f_d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 scale=0.001 0.001 0.001
- link rh_rfknuckle: geometry collision cylinder length=0.014 radius=0.007; visual mesh filename=package://sr_description/meshes/components/f_knuckle/f_knuc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 scale=0.001 0.001 0.001
- link rh_rfmiddle: geometry collision cylinder length=0.025 radius=0.007; collision sphere radius=0.007
- link rh_rfproximal: geometry collision cylinder length=0.040 radius=0.007; visual mesh filename=package://sr_description/meshes/components/f_proximal/f_pro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 scale=0.001 0.001 0.001
- link rh_thdistal: geometry collision mesh filename=package://sr_description/meshes/components/th_distal/pst/th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 scale=0.001 0.001 0.001; visual mesh filename=package://sr_description/meshes/components/th_distal/pst/th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 scale=0.001 0.001 0.001
- link rh_thmiddle: geometry collision cylinder length=0.018 radius=0.011; collision sphere radius=0.011
- link rh_thproximal: geometry collision cylinder length=0.018 radius=0.012; visual mesh filename=package://sr_description/meshes/components/th_proximal/th_p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 scale=0.001 0.001 0.001
- link rh_wrist: mass None -> 0.1; geometry collision box size=0.027 0.018 0.010; collision box size=0.027 0.018 0.010

Commit message: m

File: urdf/sr_hand_bimanual.urdf (robot description, URDF)
Before this commit: robot bimanual_shadowhand_motor, 65 links, 64 joints
Links:
- link lh_thdistal: mass None -> 0.016
- link lh_thmiddle: mass None -> 0.020
- link lh_thtip: mass None -> 0.001
- link rh_forearm: mass None -> 3.0

Commit message: updated urdf to fix mesh loading

File: urdf/sr_hand_bimanual.urdf (robot description, URDF)
Before this commit: robot bimanual_shadowhand_motor, 65 links, 64 joints
Links:
- link lh_ffdistal: geometry collision mesh filename=file://$(find botdylan)/meshes/f_distal_pst.dae scale=0.001 0.001 0.001; visual mesh filename=file://$(find botdylan)/meshes/pst/f_distal_pst.dae scale=0.001 0.001 0.001
- link lh_ffknuckle: geometry collision cylinder length=0.014 radius=0.007; visual mesh filename=file://$(find botdylan)/meshes/f_knuckle_E3M5.dae scale=0.001 0.001 0.001
- link lh_ffmiddle: geometry collision cylinder length=0.025 radius=0.007; collision sphere radius=0.007
- link lh_ffproximal: geometry collision cylinder length=0.040 radius=0.007; visual mesh filename=file://$(find botdylan)/meshes/f_proximal_E3M5.dae scale=0.001 0.001 0.001
- link lh_forearm: geometry collision box size=0.07 0.07 0.07; collision mesh filename=file://$(find botdylan)/meshes/forearm_collision_E3M5.dae scale=0.001 0.001 0.001
- link lh_lfdistal: geometry collision mesh filename=file://$(find botdylan)/meshes/f_distal_pst.dae scale=0.001 0.001 0.001; visual mesh filename=file://$(find botdylan)/meshes/f_distal_pst.dae scale=0.001 0.001 0.001
- link lh_lfknuckle: geometry collision cylinder length=0.014 radius=0.007; visual mesh filename=file://$(find botdylan)/meshes/f_knuckle_E3M5.dae scale=0.001 0.001 0.001
- link lh_lfmetacarpal: geometry collision box size=0.018 0.024 0.040; visual mesh filename=file://$(find botdylan)/meshes/lf_metacarpal_E3M5.dae scale=-0.001 0.001 0.001
- link lh_lfmiddle: geometry collision cylinder length=0.025 radius=0.007; collision sphere radius=0.007
- link lh_lfproximal: geometry collision cylinder length=0.040 radius=0.007; visual mesh filename=file://$(find botdylan)/meshes/f_proximal_E3M5.dae scale=0.001 0.001 0.001
- link lh_mfdistal: geometry collision mesh filename=file://$(find botdylan)/meshes/f_distal_pst.dae scale=0.001 0.001 0.001; visual mesh filename=file://$(find botdylan)/meshes/f_distal_pst.dae scale=0.001 0.001 0.001
- link lh_mfknuckle: geometry collision cylinder length=0.014 radius=0.007; visual mesh filename=file://$(find botdylan)/meshes/f_knuckle_E3M5.dae scale=0.001 0.001 0.001
- link lh_mfmiddle: geometry collision cylinder length=0.025 radius=0.007; collision sphere radius=0.007
- link lh_mfproximal: geometry collision cylinder length=0.040 radius=0.007; visual mesh filename=file://$(find botdylan)/meshes/f_proximal_E3M5.dae scale=0.001 0.001 0.001
- link lh_palm: geometry collision box size=0.018 0.024 0.004; collision box size=0.020 0.024 0.040
- link lh_rfdistal: geometry collision mesh filename=file://$(find botdylan)/meshes/f_distal_pst.dae scale=0.001 0.001 0.001; visual mesh filename=file://$(find botdylan)/meshes/f_distal_pst.dae scale=0.001 0.001 0.001
- link lh_rfknuckle: geometry collision cylinder length=0.014 radius=0.007; visual mesh filename=file://$(find botdylan)/meshes/f_knuckle_E3M5.dae scale=0.001 0.001 0.001
- link lh_rfmiddle: geometry collision cylinder length=0.025 radius=0.007; collision sphere radius=0.007
- link lh_rfproximal: geometry collision cylinder length=0.040 radius=0.007; visual mesh filename=file://$(find botdylan)/meshes/f_proximal_E3M5.dae scale=0.001 0.001 0.001
- link lh_thdistal: geometry collision mesh filename=file://$(find botdylan)/meshes/th_distal_pst.dae scale=0.001 0.001 0.001; visual mesh filename=file://$(find botdylan)/meshes/th_distal_pst.dae scale=0.001 0.001 0.001
- link lh_thmiddle: geometry collision cylinder length=0.018 radius=0.011; collision sphere radius=0.011
- link lh_thproximal: geometry collision cylinder length=0.018 radius=0.012; visual mesh filename=file://$(find botdylan)/meshes/th_proximal_E3M5.dae scale=0.001 0.001 0.001
- link lh_wrist: geometry collision box size=0.027 0.018 0.010; collision box size=0.027 0.018 0.010
- link rh_ffdistal: geometry collision mesh filename=file://$(find botdylan)/meshes/f_distal_pst.dae scale=0.001 0.001 0.001; visual mesh filename=file://$(find botdylan)/meshes/f_distal_pst.dae scale=0.001 0.001 0.001
- link rh_ffknuckle: geometry collision cylinder length=0.014 radius=0.007; visual mesh filename=file://$(find botdylan)/meshes/f_knuckle_E3M5.dae scale=0.001 0.001 0.001
- link rh_ffmiddle: geometry collision cylinder length=0.025 radius=0.007; collision sphere radius=0.007
- link rh_ffproximal: geometry collision cylinder length=0.040 radius=0.007; visual mesh filename=file://$(find botdylan)/meshes/f_proximal_E3M5.dae scale=0.001 0.001 0.001
- link rh_forearm: geometry collision box size=0.07 0.07 0.07; collision mesh filename=file://$(find botdylan)/meshes/forearm_collision_E3M5.dae scale=0.001 0.001 0.001
- link rh_lfdistal: geometry collision mesh filename=file://$(find botdylan)/meshes/f_distal_pst.dae scale=0.001 0.001 0.001; visual mesh filename=file://$(find botdylan)/meshes/f_distal_pst.dae scale=0.001 0.001 0.001
- link rh_lfknuckle: geometry collision cylinder length=0.014 radius=0.007; visual mesh filename=file://$(find botdylan)/meshes/f_knuckle_E3M5.dae scale=0.001 0.001 0.001
- link rh_lfmetacarpal: geometry collision box size=0.018 0.024 0.040; visual mesh filename=file://$(find botdylan)/meshes/lf_metacarpal_E3M5.dae scale=0.001 0.001 0.001
- link rh_lfmiddle: geometry collision cylinder length=0.025 radius=0.007; collision sphere radius=0.007
- link rh_lfproximal: geometry collision cylinder length=0.040 radius=0.007; visual mesh filename=file://$(find botdylan)/meshes/f_proximal_E3M5.dae scale=0.001 0.001 0.001
- link rh_mfdistal: geometry collision mesh filename=file://$(find botdylan)/meshes/f_distal_pst.dae scale=0.001 0.001 0.001; visual mesh filename=file://$(find botdylan)/meshes/f_distal_pst.dae scale=0.001 0.001 0.001
- link rh_mfknuckle: geometry collision cylinder length=0.014 radius=0.007; visual mesh filename=file://$(find botdylan)/meshes/f_knuckle_E3M5.dae scale=0.001 0.001 0.001
- link rh_mfmiddle: geometry collision cylinder length=0.025 radius=0.007; collision sphere radius=0.007
- link rh_mfproximal: geometry collision cylinder length=0.040 radius=0.007; visual mesh filename=file://$(find botdylan)/meshes/f_proximal_E3M5.dae scale=0.001 0.001 0.001
- link rh_palm: geometry collision box size=0.018 0.024 0.004; collision box size=0.020 0.024 0.040
- link rh_rfdistal: geometry collision mesh filename=file://$(find botdylan)/meshes/f_distal_pst.dae scale=0.001 0.001 0.001; visual mesh filename=file://$(find botdylan)/meshes/f_distal_pst.dae scale=0.001 0.001 0.001
- link rh_rfknuckle: geometry collision cylinder length=0.014 radius=0.007; visual mesh filename=file://$(find botdylan)/meshes/f_knuckle_E3M5.dae scale=0.001 0.001 0.001
- link rh_rfmiddle: geometry collision cylinder length=0.025 radius=0.007; collision sphere radius=0.007
- link rh_rfproximal: geometry collision cylinder length=0.040 radius=0.007; visual mesh filename=file://$(find botdylan)/meshes/f_proximal_E3M5.dae scale=0.001 0.001 0.001
- link rh_thdistal: geometry collision mesh filename=file://$(find botdylan)/meshes/th_distal_pst.dae scale=0.001 0.001 0.001; visual mesh filename=file://$(find botdylan)/meshes/th_distal_pst.dae scale=0.001 0.001 0.001
- link rh_thmiddle: geometry collision cylinder length=0.018 radius=0.011; collision sphere radius=0.011
- link rh_thproximal: geometry collision cylinder length=0.018 radius=0.012; visual mesh filename=file://$(find botdylan)/meshes/th_proximal_E3M5.dae scale=0.001 0.001 0.001
- link rh_wrist: geometry collision box size=0.027 0.018 0.010; collision box size=0.027 0.018 0.010
