Commit message: Updated guitar neck

File: urdf/guitar.urdf (robot description, URDF)
Before this commit: robot guitar_neck, 2 links, 1 joints
Links:
- added link string1; collision cylinder length=1.2 radius=0.01; visual cylinder length=1.2 radius=0.01
- link neck: geometry collision box size=0.50 1.2 0.05; visual box size=0.50 1.2 0.05
Joints:
- added joint string1_to_neck: type fixed, parent neck, child string1, origin xyz=0.00 0.00 0.05 rpy=0 0 0

Commit message: resizing guitar

File: urdf/guitar.urdf (robot description, URDF)
Before this commit: robot guitar_neck, 3 links, 2 joints
Links:
- link neck: geometry collision box size=0.10 1.5 0.02; visual box size=0.10 1.5 0.02
- link string1: geometry collision cylinder length=1.5 radius=0.002; visual cylinder length=1.5 radius=0.002
Joints:
- joint string1_to_neck: origin xyz=0.00 0.00 0.05 rpy=0 0 0 -> xyz=0.00 0.00 0.005 rpy=0 0 0

Commit message: resizing guitar

File: urdf/guitar.urdf (robot description, URDF)
Before this commit: robot guitar_neck, 3 links, 2 joints
Joints:
- joint neck_to_world: origin xyz=0.00 0.00 0.00 rpy=0 0 0 -> xyz=0.00 0.00 0.00 rpy=-1.57 1.57 0
- joint string1_to_neck: origin xyz=0.00 0.00 0.005 rpy=0 0 0 -> xyz=0.0375 0.00 0.005 rpy=0 0 0

Commit message: resizing guitar

File: urdf/guitar.urdf (robot description, URDF)
Before this commit: robot guitar_neck, 3 links, 2 joints
Joints:
- joint neck_to_world: origin xyz=0.00 0.00 0.00 rpy=-1.57 1.57 0 -> xyz=0.00 0.05 0.25 rpy=1.57 1.57 0

Commit message: fixing strings

File: urdf/guitar.urdf (robot description, URDF)
Before this commit: robot guitar_neck, 3 links, 2 joints
Links:
- removed link string1
- added link str_b; collision cylinder length=1.5 radius=0.002; visual cylinder length=1.5 radius=0.002
- added link str_high_e; collision cylinder length=1.5 radius=0.002; visual cylinder length=1.5 radius=0.002
Joints:
- added joint high_e_to_b: type fixed, parent str_high_e, child str_b, origin xyz=0.0375 0.00 0.005 rpy=0 0 0
- joint string1_to_neck: child string1 -> str_high_e

Commit message: fixing strings

File: urdf/guitar.urdf (robot description, URDF)
Before this commit: robot guitar_neck, 4 links, 3 joints
Joints:
- joint high_e_to_b: origin xyz=0.0375 0.00 0.005 rpy=0 0 0 -> xyz=0.0 0.0 0.00 rpy=0 0 0

Commit message: fixing strings

File: urdf/guitar.urdf (robot description, URDF)
Before this commit: robot guitar_neck, 4 links, 3 joints
Links:
- added link str_a; collision cylinder length=1.5 radius=0.002; visual cylinder length=1.5 radius=0.002
- added link str_d; collision cylinder length=1.5 radius=0.002; visual cylinder length=1.5 radius=0.002
- added link str_g; collision cylinder length=1.5 radius=0.002; visual cylinder length=1.5 radius=0.002
- added link str_low_e; collision cylinder length=1.5 radius=0.002; visual cylinder length=1.5 radius=0.002
Joints:
- added joint a_to_low_e: type fixed, parent str_a, child str_low_e, origin xyz=0.0 0.0 0.00 rpy=0 0 0
- added joint b_to_g: type fixed, parent str_b, child str_g, origin xyz=0.0 0.0 0.00 rpy=0 0 0
- added joint d_to_a: type fixed, parent str_d, child str_a, origin xyz=0.0 0.0 0.00 rpy=0 0 0
- added joint g_to_d: type fixed, parent str_g, child str_d, origin xyz=0.0 0.0 0.00 rpy=0 0 0

Commit message: fixing strings

File: urdf/guitar.urdf (robot description, URDF)
Before this commit: robot guitar_neck, 8 links, 7 joints
Links:
- removed link str_a
- removed link str_d
- removed link str_g
- removed link str_low_e
Joints:
- removed joint a_to_low_e
- removed joint b_to_g
- removed joint d_to_a
- removed joint g_to_d
- joint high_e_to_b: origin xyz=0.0 0.0 0.00 rpy=0 0 0 -> xyz=-0.0125 0.0 0.00 rpy=0 0 0

Commit message: fixing strings

File: urdf/guitar.urdf (robot description, URDF)
Before this commit: robot guitar_neck, 4 links, 3 joints
Joints:
- joint high_e_to_b: origin xyz=-0.0125 0.0 0.00 rpy=0 0 0 -> xyz=-0.0125 0.0 0.005 rpy=0 0 0

Commit message: fixing strings

File: urdf/guitar.urdf (robot description, URDF)
Before this commit: robot guitar_neck, 4 links, 3 joints
Links:
- added link str_a; collision cylinder length=1.5 radius=0.002; visual cylinder length=1.5 radius=0.002
- added link str_d; collision cylinder length=1.5 radius=0.002; visual cylinder length=1.5 radius=0.002
- added link str_g; collision cylinder length=1.5 radius=0.002; visual cylinder length=1.5 radius=0.002
- added link str_low_e; collision cylinder length=1.5 radius=0.002; visual cylinder length=1.5 radius=0.002
Joints:
- added joint a_to_low_e: type fixed, parent str_a, child str_low_e, origin xyz=-0.0125 0.0 0.005 rpy=0 0 0
- added joint b_to_g: type fixed, parent str_b, child str_g, origin xyz=-0.0125 0.0 0.005 rpy=0 0 0
- added joint d_to_a: type fixed, parent str_d, child str_a, origin xyz=-0.0125 0.0 0.005 rpy=0 0 0
- added joint g_to_d: type fixed, parent str_g, child str_d, origin xyz=-0.0125 0.0 0.005 rpy=0 0 0

Commit message: fixing strings

File: urdf/guitar.urdf (robot description, URDF)
Before this commit: robot guitar_neck, 8 links, 7 joints
Joints:
- joint a_to_low_e: origin xyz=-0.0125 0.0 0.005 rpy=0 0 0 -> xyz=-0.0143 0.0 0.00 rpy=0 0 0
- joint b_to_g: origin xyz=-0.0125 0.0 0.005 rpy=0 0 0 -> xyz=-0.0143 0.0 0.00 rpy=0 0 0
- joint d_to_a: origin xyz=-0.0125 0.0 0.005 rpy=0 0 0 -> xyz=-0.0143 0.0 0.00 rpy=0 0 0
- joint g_to_d: origin xyz=-0.0125 0.0 0.005 rpy=0 0 0 -> xyz=-0.0143 0.0 0.005 rpy=0 0 0
- joint high_e_to_b: origin xyz=-0.0125 0.0 0.005 rpy=0 0 0 -> xyz=-0.0143 0.0 0.005 rpy=0 0 0
- joint string1_to_neck: origin xyz=0.0375 0.00 0.005 rpy=0 0 0 -> xyz=0.0357 0.00 0.005 rpy=0 0 0

Commit message: adding frets

File: urdf/guitar.urdf (robot description, URDF)
Before this commit: robot guitar_neck, 8 links, 7 joints
Links:
- added link fret0; collision cylinder length=.1 radius=0.002; visual cylinder length=.1 radius=0.002
Joints:
- removed joint string1_to_neck
- added joint high_e_to_neck: type fixed, parent neck, child str_high_e, origin xyz=0.0357 0.00 0.005 rpy=0 0 0
- added joint neck_to_fret0: type fixed, parent neck, child fret0, origin xyz=0.0 0.75 0.003 rpy=0 0 0
- joint g_to_d: origin xyz=-0.0143 0.0 0.005 rpy=0 0 0 -> xyz=-0.0143 0.0 0.00 rpy=0 0 0

Commit message: adding frets

File: urdf/guitar.urdf (robot description, URDF)
Before this commit: robot guitar_neck, 9 links, 8 joints
Links:
- added link fret1; collision cylinder length=.1 radius=0.002; visual cylinder length=.1 radius=0.002
Joints:
- added joint fret0_to_fret1: type fixed, parent fret0, child fret1, origin xyz=0.0 -0.075 0.00 rpy=0 0 0
- joint neck_to_fret0: origin xyz=0.0 0.75 0.003 rpy=0 0 0 -> xyz=0.0 0.75 0.005 rpy=0 0 0

Commit message: adding frets

File: urdf/guitar.urdf (robot description, URDF)
Before this commit: robot guitar_neck, 10 links, 9 joints
Joints:
- joint fret0_to_fret1: origin xyz=0.0 -0.075 0.00 rpy=0 0 0 -> xyz=0.0 -0.075 0.0 rpy=0 0 0
- joint high_e_to_b: origin xyz=-0.0143 0.0 0.005 rpy=0 0 0 -> xyz=-0.0143 0.0 0.000 rpy=0 0 0
- joint high_e_to_neck: origin xyz=0.0357 0.00 0.005 rpy=0 0 0 -> xyz=0.0357 0.00 0.01 rpy=0 0 0
- joint neck_to_fret0: origin xyz=0.0 0.75 0.005 rpy=0 0 0 -> xyz=0.0 0.75 0.01 rpy=0 0 0

Commit message: adding frets

File: urdf/guitar.urdf (robot description, URDF)
Before this commit: robot guitar_neck, 10 links, 9 joints
Links:
- added link fret10; collision cylinder length=.1 radius=0.002; visual cylinder length=.1 radius=0.002
- added link fret11; collision cylinder length=.1 radius=0.002; visual cylinder length=.1 radius=0.002
- added link fret12; collision cylinder length=.1 radius=0.002; visual cylinder length=.1 radius=0.002
- added link fret13; collision cylinder length=.1 radius=0.002; visual cylinder length=.1 radius=0.002
- added link fret14; collision cylinder length=.1 radius=0.002; visual cylinder length=.1 radius=0.002
- added link fret15; collision cylinder length=.1 radius=0.002; visual cylinder length=.1 radius=0.002
- added link fret16; collision cylinder length=.1 radius=0.002; visual cylinder length=.1 radius=0.002
- added link fret17; collision cylinder length=.1 radius=0.002; visual cylinder length=.1 radius=0.002
- added link fret18; collision cylinder length=.1 radius=0.002; visual cylinder length=.1 radius=0.002
- added link fret19; collision cylinder length=.1 radius=0.002; visual cylinder length=.1 radius=0.002
- added link fret2; collision cylinder length=.1 radius=0.002; visual cylinder length=.1 radius=0.002
- added link fret20; collision cylinder length=.1 radius=0.002; visual cylinder length=.1 radius=0.002
- added link fret3; collision cylinder length=.1 radius=0.002; visual cylinder length=.1 radius=0.002
- added link fret4; collision cylinder length=.1 radius=0.002; visual cylinder length=.1 radius=0.002
- added link fret5; collision cylinder length=.1 radius=0.002; visual cylinder length=.1 radius=0.002
- added link fret6; collision cylinder length=.1 radius=0.002; visual cylinder length=.1 radius=0.002
- added link fret7; collision cylinder length=.1 radius=0.002; visual cylinder length=.1 radius=0.002
- added link fret8; collision cylinder length=.1 radius=0.002; visual cylinder length=.1 radius=0.002
- added link fret9; collision cylinder length=.1 radius=0.002; visual cylinder length=.1 radius=0.002
Joints:
- added joint fret10_to_fret11: type fixed, parent fret10, child fret11, origin xyz=0.0 -0.075 0.0 rpy=0 0 0
- added joint fret11_to_fret12: type fixed, parent fret11, child fret12, origin xyz=0.0 -0.075 0.0 rpy=0 0 0
- added joint fret12_to_fret13: type fixed, parent fret12, child fret13, origin xyz=0.0 -0.075 0.0 rpy=0 0 0
- added joint fret13_to_fret14: type fixed, parent fret13, child fret14, origin xyz=0.0 -0.075 0.0 rpy=0 0 0
- added joint fret14_to_fret15: type fixed, parent fret14, child fret15, origin xyz=0.0 -0.075 0.0 rpy=0 0 0
- added joint fret15_to_fret16: type fixed, parent fret15, child fret16, origin xyz=0.0 -0.075 0.0 rpy=0 0 0
- added joint fret16_to_fret17: type fixed, parent fret16, child fret17, origin xyz=0.0 -0.075 0.0 rpy=0 0 0
- added joint fret17_to_fret18: type fixed, parent fret17, child fret18, origin xyz=0.0 -0.075 0.0 rpy=0 0 0
- added joint fret18_to_fret19: type fixed, parent fret18, child fret19, origin xyz=0.0 -0.075 0.0 rpy=0 0 0
- added joint fret19_to_fret20: type fixed, parent fret19, child fret20, origin xyz=0.0 -0.075 0.0 rpy=0 0 0
- added joint fret1_to_fret2: type fixed, parent fret1, child fret2, origin xyz=0.0 -0.075 0.0 rpy=0 0 0
- added joint fret2_to_fret3: type fixed, parent fret2, child fret3, origin xyz=0.0 -0.075 0.0 rpy=0 0 0
- added joint fret3_to_fret4: type fixed, parent fret3, child fret4, origin xyz=0.0 -0.075 0.0 rpy=0 0 0
- added joint fret4_to_fret5: type fixed, parent fret4, child fret5, origin xyz=0.0 -0.075 0.0 rpy=0 0 0
- added joint fret5_to_fret6: type fixed, parent fret5, child fret6, origin xyz=0.0 -0.075 0.0 rpy=0 0 0
- added joint fret6_to_fret7: type fixed, parent fret6, child fret7, origin xyz=0.0 -0.075 0.0 rpy=0 0 0
- added joint fret7_to_fret8: type fixed, parent fret7, child fret8, origin xyz=0.0 -0.075 0.0 rpy=0 0 0
- added joint fret8_to_fret9: type fixed, parent fret8, child fret9, origin xyz=0.0 -0.075 0.0 rpy=0 0 0
- added joint fret9_to_fret10: type fixed, parent fret9, child fret10, origin xyz=0.0 -0.075 0.0 rpy=0 0 0

Commit message: adding strumbox

File: urdf/guitar.urdf (robot description, URDF)
Before this commit: robot guitar_neck, 29 links, 28 joints
Links:
- added link strum_cylinder; collision cylinder length=0.02 radius=0.075; visual cylinder length=0.02 radius=0.075
Joints:
- added joint strum_to_guitar: type fixed, parent neck, child strum_cylinder, origin xyz=0.05 -0.825 0.02 rpy=0 0 0

Commit message: adding strumbox

File: urdf/guitar.urdf (robot description, URDF)
Before this commit: robot guitar_neck, 30 links, 29 joints
Links:
- link strum_cylinder: geometry collision cylinder length=0.02 radius=0.075; visual cylinder length=0.02 radius=0.1
Joints:
- joint strum_to_guitar: origin xyz=0.05 -0.825 0.02 rpy=0 0 0 -> xyz=0.0 -1 0.0 rpy=0 0 0

Commit message: adding strumbox

File: urdf/guitar.urdf (robot description, URDF)
Before this commit: robot guitar_neck, 30 links, 29 joints
Links:
- link str_a: geometry collision cylinder length=1.7 radius=0.002; visual cylinder length=1.7 radius=0.002
- link str_b: geometry collision cylinder length=1.7 radius=0.002; visual cylinder length=1.7 radius=0.002
- link str_d: geometry collision cylinder length=1.7 radius=0.002; visual cylinder length=1.7 radius=0.002
- link str_g: geometry collision cylinder length=1.7 radius=0.002; visual cylinder length=1.7 radius=0.002
- link str_high_e: geometry collision cylinder length=1.7 radius=0.002; visual cylinder length=1.7 radius=0.002
- link str_low_e: geometry collision cylinder length=1.7 radius=0.002; visual cylinder length=1.7 radius=0.002
- link strum_cylinder: geometry collision cylinder length=0.02 radius=0.1; visual cylinder length=0.02 radius=0.1
Joints:
- joint strum_to_guitar: origin xyz=0.0 -1 0.0 rpy=0 0 0 -> xyz=0.0 -0.85 0.0 rpy=0 0 0

Commit message: adding strumbox

File: urdf/guitar.urdf (robot description, URDF)
Before this commit: robot guitar_neck, 30 links, 29 joints
Links:
- link str_a: geometry collision cylinder length=1.85 radius=0.002; visual cylinder length=1.85 radius=0.002
- link str_b: geometry collision cylinder length=1.85 radius=0.002; visual cylinder length=1.85 radius=0.002
- link str_d: geometry collision cylinder length=1.85 radius=0.002; visual cylinder length=1.85 radius=0.002
- link str_g: geometry collision cylinder length=1.85 radius=0.002; visual cylinder length=1.85 radius=0.002
- link str_high_e: geometry collision cylinder length=1.85 radius=0.002; visual cylinder length=1.85 radius=0.002
- link str_low_e: geometry collision cylinder length=1.85 radius=0.002; visual cylinder length=1.85 radius=0.002
Joints:
- joint strum_to_guitar: origin xyz=0.0 -0.85 0.0 rpy=0 0 0 -> xyz=0.0 -0.825 0.0 rpy=0 0 0

Commit message: repositioning guitar

File: urdf/guitar.urdf (robot description, URDF)
Before this commit: robot guitar_neck, 30 links, 29 joints
Joints:
- joint neck_to_world: origin xyz=0.00 0.05 0.25 rpy=1.57 1.57 0 -> xyz=0.00 -0.05 0.25 rpy=-1.57 1.57 0

Commit message: repositioning strings

File: urdf/guitar.urdf (robot description, URDF)
Before this commit: robot guitar_neck, 30 links, 29 joints
Links:
- link str_a: geometry collision cylinder length=1.65 radius=0.002; visual cylinder length=1.65 radius=0.002
- link str_b: geometry collision cylinder length=1.65 radius=0.002; visual cylinder length=1.65 radius=0.002
- link str_d: geometry collision cylinder length=1.65 radius=0.002; visual cylinder length=1.65 radius=0.002
- link str_g: geometry collision cylinder length=1.65 radius=0.002; visual cylinder length=1.65 radius=0.002
- link str_high_e: geometry collision cylinder length=1.65 radius=0.002; visual cylinder length=1.65 radius=0.002
- link str_low_e: geometry collision cylinder length=1.65 radius=0.002; visual cylinder length=1.65 radius=0.002
Joints:
- joint high_e_to_neck: origin xyz=0.0357 0.00 0.01 rpy=0 0 0 -> xyz=0.0357 -0.1 0.01 rpy=0 0 0

Commit message: repositioning strings

File: urdf/guitar.urdf (robot description, URDF)
Before this commit: robot guitar_neck, 30 links, 29 joints
Links:
- link str_a: geometry collision cylinder length=1.7 radius=0.002; visual cylinder length=1.7 radius=0.002
- link str_b: geometry collision cylinder length=1.7 radius=0.002; visual cylinder length=1.7 radius=0.002
- link str_d: geometry collision cylinder length=1.7 radius=0.002; visual cylinder length=1.7 radius=0.002
- link str_g: geometry collision cylinder length=1.7 radius=0.002; visual cylinder length=1.7 radius=0.002
- link str_high_e: geometry collision cylinder length=1.7 radius=0.002; visual cylinder length=1.7 radius=0.002
- link str_low_e: geometry collision cylinder length=1.7 radius=0.002; visual cylinder length=1.7 radius=0.002
Joints:
- joint high_e_to_neck: origin xyz=0.0357 -0.1 0.01 rpy=0 0 0 -> xyz=0.0357 -0.075 0.01 rpy=0 0 0

Commit message: repositioning strings

File: urdf/guitar.urdf (robot description, URDF)
Before this commit: robot guitar_neck, 30 links, 29 joints
Joints:
- joint high_e_to_neck: origin xyz=0.0357 -0.075 0.01 rpy=0 0 0 -> xyz=0.0357 -0.0875 0.01 rpy=0 0 0

Commit message: repositioning strings

File: urdf/guitar.urdf (robot description, URDF)
Before this commit: robot guitar_neck, 30 links, 29 joints
Links:
- link str_a: geometry collision cylinder length=1.675 radius=0.002; visual cylinder length=1.675 radius=0.002
- link str_b: geometry collision cylinder length=1.675 radius=0.002; visual cylinder length=1.675 radius=0.002
- link str_d: geometry collision cylinder length=1.675 radius=0.002; visual cylinder length=1.675 radius=0.002
- link str_g: geometry collision cylinder length=1.675 radius=0.002; visual cylinder length=1.675 radius=0.002
- link str_high_e: geometry collision cylinder length=1.675 radius=0.002; visual cylinder length=1.675 radius=0.002
- link str_low_e: geometry collision cylinder length=1.675 radius=0.002; visual cylinder length=1.675 radius=0.002

Commit message: repositioning GUITAR

File: urdf/guitar.urdf (robot description, URDF)
Before this commit: robot guitar_neck, 30 links, 29 joints
Joints:
- joint neck_to_world: origin xyz=0.00 -0.05 0.25 rpy=-1.57 1.57 0 -> xyz=0.00 -0.025 0.3 rpy=-1.57 1.57 0

Commit message: repositioning strings

File: urdf/guitar.urdf (robot description, URDF)
Before this commit: robot guitar_neck, 30 links, 29 joints
Joints:
- joint neck_to_world: origin xyz=0.00 -0.025 0.3 rpy=-1.57 1.57 0 -> xyz=0.00 -0.04 0.3 rpy=-1.57 1.57 0

Commit message: fret width changed to .05

File: urdf/guitar.urdf (robot description, URDF)
Before this commit: robot guitar_neck, 30 links, 29 joints
Joints:
- joint fret0_to_fret1: origin xyz=0.0 -0.075 0.0 rpy=0 0 0 -> xyz=0.0 -0.050 0.0 rpy=0 0 0
- joint fret10_to_fret11: origin xyz=0.0 -0.075 0.0 rpy=0 0 0 -> xyz=0.0 -0.050 0.0 rpy=0 0 0
- joint fret11_to_fret12: origin xyz=0.0 -0.075 0.0 rpy=0 0 0 -> xyz=0.0 -0.050 0.0 rpy=0 0 0
- joint fret12_to_fret13: origin xyz=0.0 -0.075 0.0 rpy=0 0 0 -> xyz=0.0 -0.050 0.0 rpy=0 0 0
- joint fret13_to_fret14: origin xyz=0.0 -0.075 0.0 rpy=0 0 0 -> xyz=0.0 -0.050 0.0 rpy=0 0 0
- joint fret14_to_fret15: origin xyz=0.0 -0.075 0.0 rpy=0 0 0 -> xyz=0.0 -0.050 0.0 rpy=0 0 0
- joint fret15_to_fret16: origin xyz=0.0 -0.075 0.0 rpy=0 0 0 -> xyz=0.0 -0.050 0.0 rpy=0 0 0
- joint fret16_to_fret17: origin xyz=0.0 -0.075 0.0 rpy=0 0 0 -> xyz=0.0 -0.050 0.0 rpy=0 0 0
- joint fret17_to_fret18: origin xyz=0.0 -0.075 0.0 rpy=0 0 0 -> xyz=0.0 -0.050 0.0 rpy=0 0 0
- joint fret18_to_fret19: origin xyz=0.0 -0.075 0.0 rpy=0 0 0 -> xyz=0.0 -0.050 0.0 rpy=0 0 0
- joint fret19_to_fret20: origin xyz=0.0 -0.075 0.0 rpy=0 0 0 -> xyz=0.0 -0.050 0.0 rpy=0 0 0
- joint fret1_to_fret2: origin xyz=0.0 -0.075 0.0 rpy=0 0 0 -> xyz=0.0 -0.050 0.0 rpy=0 0 0
- joint fret2_to_fret3: origin xyz=0.0 -0.075 0.0 rpy=0 0 0 -> xyz=0.0 -0.050 0.0 rpy=0 0 0
- joint fret3_to_fret4: origin xyz=0.0 -0.075 0.0 rpy=0 0 0 -> xyz=0.0 -0.050 0.0 rpy=0 0 0
- joint fret4_to_fret5: origin xyz=0.0 -0.075 0.0 rpy=0 0 0 -> xyz=0.0 -0.050 0.0 rpy=0 0 0
- joint fret5_to_fret6: origin xyz=0.0 -0.075 0.0 rpy=0 0 0 -> xyz=0.0 -0.050 0.0 rpy=0 0 0
- joint fret6_to_fret7: origin xyz=0.0 -0.075 0.0 rpy=0 0 0 -> xyz=0.0 -0.050 0.0 rpy=0 0 0
- joint fret7_to_fret8: origin xyz=0.0 -0.075 0.0 rpy=0 0 0 -> xyz=0.0 -0.050 0.0 rpy=0 0 0
- joint fret8_to_fret9: origin xyz=0.0 -0.075 0.0 rpy=0 0 0 -> xyz=0.0 -0.050 0.0 rpy=0 0 0
- joint fret9_to_fret10: origin xyz=0.0 -0.075 0.0 rpy=0 0 0 -> xyz=0.0 -0.050 0.0 rpy=0 0 0

Commit message: moved guitar around

File: urdf/guitar.urdf (robot description, URDF)
Before this commit: robot guitar_neck, 30 links, 29 joints
Joints:
- joint neck_to_world: origin xyz=0.00 -0.04 0.3 rpy=-1.57 1.57 0 -> xyz=0.00 0.2 0.1 rpy=0 0 1.57

Commit message: updated guitar pos

File: urdf/guitar.urdf (robot description, URDF)
Before this commit: robot guitar_neck, 30 links, 29 joints
Joints:
- joint neck_to_world: origin xyz=0.00 0.2 0.1 rpy=0 0 1.57 -> xyz=-0.5 0.3 0.1 rpy=0 0 1.57

Commit message: updated guitar pos

File: urdf/guitar.urdf (robot description, URDF)
Before this commit: robot guitar_neck, 30 links, 29 joints
Joints:
- joint neck_to_world: origin xyz=-0.5 0.3 0.1 rpy=0 0 1.57 -> xyz=-0.5 0.225 0.1 rpy=0 0 1.57

Commit message: updated guitar pos

File: urdf/guitar.urdf (robot description, URDF)
Before this commit: robot guitar_neck, 30 links, 29 joints
Joints:
- joint neck_to_world: origin xyz=-0.5 0.225 0.1 rpy=0 0 1.57 -> xyz=-1 0.325 0.1 rpy=0 0 1.57

Commit message: updated guitar pos

File: urdf/guitar.urdf (robot description, URDF)
Before this commit: robot guitar_neck, 30 links, 29 joints
Joints:
- joint neck_to_world: origin xyz=-1 0.325 0.1 rpy=0 0 1.57 -> xyz=-.9 0.35 0.075 rpy=0 0 1.57

Commit message: updated guitar pos

File: urdf/guitar.urdf (robot description, URDF)
Before this commit: robot guitar_neck, 30 links, 29 joints
Joints:
- joint neck_to_world: origin xyz=-.9 0.35 0.075 rpy=0 0 1.57 -> xyz=-.8 0.375 0.08 rpy=0 0 1.57

Commit message: updated guitar pos

File: urdf/guitar.urdf (robot description, URDF)
Before this commit: robot guitar_neck, 30 links, 29 joints
Joints:
- joint neck_to_world: origin xyz=-.8 0.375 0.08 rpy=0 0 1.57 -> xyz=-.8 0.375 0.095 rpy=0 0 1.57

Commit message: updated str pos

File: urdf/guitar.urdf (robot description, URDF)
Before this commit: robot guitar_neck, 30 links, 29 joints
Joints:
- joint a_to_low_e: origin xyz=-0.0143 0.0 0.00 rpy=0 0 0 -> xyz=-0.0075 0.0 0.00 rpy=0 0 0
- joint b_to_g: origin xyz=-0.0143 0.0 0.00 rpy=0 0 0 -> xyz=-0.0075 0.0 0.00 rpy=0 0 0
- joint d_to_a: origin xyz=-0.0143 0.0 0.00 rpy=0 0 0 -> xyz=-0.0075 0.0 0.00 rpy=0 0 0
- joint g_to_d: origin xyz=-0.0143 0.0 0.00 rpy=0 0 0 -> xyz=-0.0075 0.0 0.00 rpy=0 0 0
- joint high_e_to_b: origin xyz=-0.0143 0.0 0.000 rpy=0 0 0 -> xyz=-0.0075 0.0 0.000 rpy=0 0 0
- joint high_e_to_neck: origin xyz=0.0357 -0.0875 0.01 rpy=0 0 0 -> xyz=0.0425 -0.0875 0.01 rpy=0 0 0
