Commit message: updated guitar pos

File: urdf/guitar.urdf (robot description, URDF)
Before this commit: robot guitar_neck, 30 links, 29 joints
Links:
- link fret0: geometry collision cylinder length=.05 radius=0.002; visual cylinder length=.05 radius=0.002
- link fret1: geometry collision cylinder length=.05 radius=0.002; visual cylinder length=.05 radius=0.002
- link fret10: geometry collision cylinder length=.05 radius=0.002; visual cylinder length=.05 radius=0.002
- link fret11: geometry collision cylinder length=.05 radius=0.002; visual cylinder length=.05 radius=0.002
- link fret12: geometry collision cylinder length=.05 radius=0.002; visual cylinder length=.05 radius=0.002
- link fret13: geometry collision cylinder length=.05 radius=0.002; visual cylinder length=.05 radius=0.002
- link fret14: geometry collision cylinder length=.05 radius=0.002; visual cylinder length=.05 radius=0.002
- link fret15: geometry collision cylinder length=.05 radius=0.002; visual cylinder length=.05 radius=0.002
- link fret16: geometry collision cylinder length=.05 radius=0.002; visual cylinder length=.05 radius=0.002
- link fret17: geometry collision cylinder length=.05 radius=0.002; visual cylinder length=.05 radius=0.002
- link fret18: geometry collision cylinder length=.05 radius=0.002; visual cylinder length=.05 radius=0.002
- link fret19: geometry collision cylinder length=.05 radius=0.002; visual cylinder length=.05 radius=0.002
- link fret2: geometry collision cylinder length=.05 radius=0.002; visual cylinder length=.05 radius=0.002
- link fret20: geometry collision cylinder length=.05 radius=0.002; visual cylinder length=.05 radius=0.002
- link fret3: geometry collision cylinder length=.05 radius=0.002; visual cylinder length=.05 radius=0.002
- link fret4: geometry collision cylinder length=.05 radius=0.002; visual cylinder length=.05 radius=0.002
- link fret5: geometry collision cylinder length=.05 radius=0.002; visual cylinder length=.05 radius=0.002
- link fret6: geometry collision cylinder length=.05 radius=0.002; visual cylinder length=.05 radius=0.002
- link fret7: geometry collision cylinder length=.05 radius=0.002; visual cylinder length=.05 radius=0.002
- link fret8: geometry collision cylinder length=.05 radius=0.002; visual cylinder length=.05 radius=0.002
- link fret9: geometry collision cylinder length=.05 radius=0.002; visual cylinder length=.05 radius=0.002
- link neck: geometry collision box size=0.05 1.5 0.015; visual box size=0.05 1.5 0.015
Joints:
- joint neck_to_fret0: origin xyz=0.0 0.75 0.01 rpy=0 0 0 -> xyz=0.025 0.75 0.01 rpy=0 0 0
- joint neck_to_world: origin xyz=-.8 0.375 0.095 rpy=0 0 1.57 -> xyz=-.75 0.245 0.115 rpy=0 0 1.57

Commit message: adjusted strum cylinder position

File: urdf/guitar.urdf (robot description, URDF)
Before this commit: robot guitar_neck, 30 links, 29 joints
Joints:
- joint strum_to_guitar: origin xyz=0.0 -0.825 0.0 rpy=0 0 0 -> xyz=0.025 -0.825 0.0 rpy=0 0 0
